Commit message: Super janky way of controlling all 4 wheels with gazebo joint controllers. Absolutely needs to be updated.

File: src/rmc_robot_model/urdf/rmc_robot_model.urdf (robot description, URDF)
Before this commit: robot rmc_robot_model, 9 links, 8 joints
Links:
- removed link conveyor
- removed link dispense
- removed link endeffector_rot
- removed link linear_trans
Joints:
- removed joint conveyor
- removed joint dis
- removed joint linact
- removed joint rackpin
- joint axle1: axis 0 0 0 -> 0 0 1; limit (none) -> effort=30 velocity=1.0; type fixed -> continuous
- joint axle2: axis 0 0 0 -> 0 0 1; limit (none) -> effort=30 velocity=1.0; type fixed -> continuous
- joint axle3: axis 0 0 0 -> 0 0 1; limit (none) -> effort=30 velocity=1.0; type fixed -> continuous
- joint axle4: axis 0 0 0 -> 0 0 1; limit (none) -> effort=30 velocity=1.0; type fixed -> continuous

Commit message: Updated robot model. Stil very broken

File: src/rmc_robot_model/urdf/rmc_robot_model.urdf (robot description, URDF)
Before this commit: robot rmc_robot_model, 5 links, 4 joints
Links:
- added link conveyor_bottom, mass 0.460858078898315; collision mesh filename=package://rmc_robot_model/meshes/conveyor_bottom.STL; visual mesh filename=package://rmc_robot_model/meshes/conveyor_bottom.STL
- added link conveyor_top, mass 0.76532; collision mesh filename=package://rmc_robot_model/meshes/conveyor_top.STL; visual mesh filename=package://rmc_robot_model/meshes/conveyor_top.STL
- added link dispense, mass 0.727785005713152; collision mesh filename=package://rmc_robot_model/meshes/dispense.STL; visual mesh filename=package://rmc_robot_model/meshes/dispense.STL
- added link endeffector_rot, mass 0.31419; collision mesh filename=package://rmc_robot_model/meshes/endeffector_rot.STL; visual mesh filename=package://rmc_robot_model/meshes/endeffector_rot.STL
- added link linear_trans, mass 0.41314; collision mesh filename=package://rmc_robot_model/meshes/linear_trans.STL; visual mesh filename=package://rmc_robot_model/meshes/linear_trans.STL
- link drivetrainbase: mass 2.0869 -> 3.9785
- link wheel1: mass 1.2142 -> 1.2253
- link wheel2: mass 1.2142 -> 1.2253
- link wheel3: mass 1.2142 -> 1.2253
- link wheel4: mass 1.2142 -> 1.2253
Joints:
- added joint conveyor: type continuous, parent linear_trans, child conveyor_top, origin xyz=0.075 0.39185 0.51933 rpy=0.6511 0 3.1416, axis -1 0 0, limit lower=0 upper=0 effort=0 velocity=0
- added joint limit_angles: type revolute, parent drivetrainbase, child endeffector_rot, origin xyz=0.38615 0 0.1082 rpy=0 0 0, axis 1 0 0, limit lower=0.384 upper=1.309 effort=0 velocity=0
- added joint rackpin: type prismatic, parent endeffector_rot, child linear_trans, origin xyz=-0.13993 0.36358 -0.065882 rpy=0.70262 0 0, axis 0 0 1, limit lower=0 upper=0.462 effort=0 velocity=0
- added joint scissor: type prismatic, parent drivetrainbase, child dispense, origin xyz=0.24486 0.00037342 0.31349 rpy=1.5708 0 1.5708, axis 0 1 0, limit lower=0 upper=0.3 effort=0 velocity=0
- added joint shaft: type continuous, parent linear_trans, child conveyor_bottom, origin xyz=0.075 0.45393 -0.37125 rpy=1.4673 0 3.1416, axis 1 0 0
- joint axle1: limit effort=30 velocity=1.0 -> (none); origin xyz=0.44561 0.1492 0.13512 rpy=1.5708 -1.2203 1.5708 -> xyz=0.44561 0.1492 0.13512 rpy=1.5708 -1.2206 1.5708
- joint axle2: limit effort=30 velocity=1.0 -> (none); origin xyz=0.047286 0.1492 0.13512 rpy=-1.5708 1.3729 1.5708 -> xyz=0.047286 0.1492 0.13512 rpy=-1.5708 0.70849 1.5708
- joint axle3: limit effort=30 velocity=1.0 -> (none)
- joint axle4: limit effort=30 velocity=1.0 -> (none)
