Commit message: Fixed joint location defintions for wheels

File: src/FullMech_Rep/urdf/FullMech_Rep.urdf (robot description, URDF)
Before this commit: robot FullMech_Rep, 9 links, 8 joints
Joints:
- joint axle2: origin xyz=0.47 0.0896 0 rpy=0 0 0 -> xyz=0.16 0.115 -0.19 rpy=0 0 0
- joint axle3: origin xyz=0.47 0.0896 0 rpy=0 0 0 -> xyz=0.78 0.115 0.19 rpy=0 0 0
- joint axle4: origin xyz=0.47 0.0896 0 rpy=0 0 0 -> xyz=0.78 0.115 -0.19 rpy=0 0 0

Commit message: Updated joint limits on newest robot model

File: src/FullMech_Rep/urdf/FullMech_Rep.urdf (robot description, URDF)
Before this commit: robot FullMech_Rep, 9 links, 8 joints
Joints:
- joint rack: limit lower=0 upper=0.5 effort=5 velocity=0.25 -> lower=-0.5 upper=0.0 effort=5 velocity=0.25
- joint scissor: limit lower=0 upper=0.5 effort=5 velocity=0.25 -> lower=-0.1 upper=0.3 effort=5 velocity=0.25

Commit message: Latest package from mechanical team. Almost everything is perfect with small issues with dump bucket

File: src/FullMech_Rep/urdf/FullMech_Rep.urdf (robot description, URDF)
Before this commit: robot FullMech_Rep, 9 links, 8 joints
Links:
- link dispense: mass 0.490259886127997 -> 0.490259886128
Joints:
- joint axle1: origin xyz=0.16 0.115 0.19 rpy=0 0 0 -> xyz=0.15 0.115 0.18271 rpy=0 0 0.70807
- joint axle2: origin xyz=0.16 0.115 -0.19 rpy=0 0 0 -> xyz=0.15 0.115 -0.18271 rpy=3.1416 0 -2.3981
- joint axle3: origin xyz=0.78 0.115 0.19 rpy=0 0 0 -> xyz=0.7 0.115 -0.18271 rpy=3.1416 0 -2.2351
- joint axle4: origin xyz=0.78 0.115 -0.19 rpy=0 0 0 -> xyz=0.7 0.115 0.18271 rpy=0 0 0.70807
- joint dispense: limit lower=0 upper=1.57 effort=5 velocity=0.25 -> lower=0 upper=1.05 effort=5 velocity=0.25; origin xyz=0.47 0.0896 0 rpy=0 0 0 -> xyz=0.175 0.27513 0 rpy=0 0 0
- joint scissor: limit lower=-0.1 upper=0.3 effort=5 velocity=0.25 -> lower=-0.1 upper=0.4 effort=5 velocity=0.25

Commit message: Mostly working differential drive implementation for the drivetrain. Has some weird physics interactions during turning possibly due to other subsystems.

File: src/FullMech_Rep/urdf/FullMech_Rep.urdf (robot description, URDF)
Before this commit: robot FullMech_Rep, 9 links, 8 joints
Links:
- link wheel1: geometry collision cylinder length=0.05 radius=.12; visual cylinder length=0.05 radius=.12
- link wheel2: geometry collision cylinder length=0.05 radius=.12; visual cylinder length=0.05 radius=.12
- link wheel3: geometry collision cylinder length=0.05 radius=.12; visual cylinder length=0.05 radius=.12
- link wheel4: geometry collision cylinder length=0.05 radius=.12; visual cylinder length=0.05 radius=.12
Joints:
- joint axle1: origin xyz=0.15 0.115 0.18271 rpy=0 0 0.70807 -> xyz=0.15 0.115 0.18271 rpy=0 3.14 0.70807
- joint axle4: origin xyz=0.7 0.115 0.18271 rpy=0 0 0.70807 -> xyz=0.7 0.115 0.18271 rpy=0 3.14 0.70807
- joint rotate: limit lower=0.384 upper=1.309 effort=5 velocity=0.25 -> lower=0.7 upper=0.8 effort=5 velocity=0.25
- joint scissor: limit lower=-0.1 upper=0.4 effort=5 velocity=0.25 -> lower=-0.1 upper=0.0 effort=5 velocity=0.25

Commit message: Lowered mass and inertia values for end effector and dispensing to stop model from exploding and launching into space

File: src/FullMech_Rep/urdf/FullMech_Rep.urdf (robot description, URDF)
Before this commit: robot FullMech_Rep, 9 links, 8 joints
Links:
- link dispense: mass 0.490259886128 -> .01
- link rotate_conv: mass 4.12035499957539 -> .01
- link storage: mass 0.248919999999999 -> .01
- link translation: mass 4.12035499957539 -> .01
Joints:
- joint scissor: limit lower=-0.1 upper=0.0 effort=5 velocity=0.25 -> lower=-0.15 upper=0.0 effort=5 velocity=0.25

Commit message: Working teleoperation of the three major subsytems in simulation. Still need to fix initial joint states.

File: src/FullMech_Rep/urdf/FullMech_Rep.urdf (robot description, URDF)
Before this commit: robot FullMech_Rep, 9 links, 8 joints
Joints:
- joint dispense: limit lower=0 upper=1.05 effort=5 velocity=0.25 -> lower=0 upper=1.05 effort=5 velocity=0.8
- joint rotate: limit lower=0.7 upper=0.8 effort=5 velocity=0.25 -> lower=0.384 upper=1.25 effort=5 velocity=0.5
- joint scissor: limit lower=-0.15 upper=0.0 effort=5 velocity=0.25 -> lower=-0.15 upper=0.3 effort=5 velocity=0.25

Commit message: Added laser scanner to robot model. Added robot state publisher node to launch file to publish transforms between drivetrain and the rest of the links

File: src/FullMech_Rep/urdf/FullMech_Rep.urdf (robot description, URDF)
Before this commit: robot FullMech_Rep, 9 links, 8 joints
Links:
- added link sensor_laser, mass 1; collision cylinder length=0.1 radius=0.05; visual cylinder length=0.05 radius=0.05
Joints:
- added joint joint_sensor_laser: type fixed, parent drivetrain, child sensor_laser, origin xyz=1.05 0.3 0.0 rpy=1.57 0.0 0.0

Commit message: Latest model from Russell to correct coordinate plane defintions. Added camera to the robot. Mapping still broken

File: src/FullMech_Rep/urdf/FullMech_Rep.urdf (robot description, URDF)
Before this commit: robot FullMech_Rep, 10 links, 9 joints
Links:
- removed link dispense
- added link camera_link, mass 1e-5; collision box size=.05 .05 .05; visual box size=.05 .05 .05
- added link dispense_rotate, mass .01; collision mesh filename=package://FullMech_Rep/meshes/dispense_rotate.STL; visual mesh filename=package://FullMech_Rep/meshes/dispense_rotate.STL
- link wheel1: mass 1.22527899288124 -> 1.22527899288125
- link wheel4: mass 1.22527899288124 -> 1.22527899288125
Joints:
- removed joint dispense
- added joint camera_joint: type continuous, parent drivetrain, child camera_link, origin xyz=0 0.2 0.45 rpy=0 0 3.14, axis 0 0 1
- added joint dispense_rotate: type revolute, parent storage, child dispense_rotate, origin xyz=0.175 0 0.42444 rpy=1.5708 0 0, axis 0 0 -1, limit lower=0 upper=1.05 effort=5 velocity=0.8
- joint axle1: origin xyz=0.15 0.115 0.18271 rpy=0 3.14 0.70807 -> xyz=0.15 -0.18271 0.115 rpy=1.5708 -0.53093 3.14
- joint axle2: origin xyz=0.15 0.115 -0.18271 rpy=3.1416 0 -2.3981 -> xyz=0.15 0.18271 0.115 rpy=1.5708 0.74348 3.1416
- joint axle3: origin xyz=0.7 0.115 -0.18271 rpy=3.1416 0 -2.2351 -> xyz=0.7 0.18271 0.115 rpy=1.5708 0.90647 3.1416
- joint axle4: origin xyz=0.7 0.115 0.18271 rpy=0 3.14 0.70807 -> xyz=0.7 -0.18271 0.115 rpy=1.5708 -0.53093 3.14
- joint joint_sensor_laser: origin xyz=1.05 0.3 0.0 rpy=1.57 0.0 0.0 -> xyz=1.05 0 0.5 rpy=0 0.0 0.0
- joint rack: axis -0.2999 0.95397 0 -> -0.2999 0 0.95397; origin xyz=-0.47 -0.0896 0 rpy=0 0 0 -> xyz=-0.0083328 -0.77093 0.1 rpy=-1.5708 0 1.2662
- joint rotate: origin xyz=0.47 0.0896 0 rpy=0 0 0 -> xyz=0.73794 0.1 0.22326 rpy=1.5708 1.2662 0
- joint scissor: axis 0 1 0 -> 0 0 1; limit lower=-0.15 upper=0.3 effort=5 velocity=0.25 -> lower=-0.3 upper=0.1 effort=5 velocity=0.25

Commit message: partially integrated tagslam into simulation

File: src/FullMech_Rep/urdf/FullMech_Rep.urdf (robot description, URDF)
Before this commit: robot FullMech_Rep, 11 links, 10 joints
Links:
- link camera_link: mass 1e-5 -> 0.000005
- link dispense_rotate: mass .01 -> .0001
- link drivetrain: mass 3.77582130485992 -> .01
- link rotate_conv: mass .01 -> .0001
- link sensor_laser: mass 1 -> .0001
- link storage: mass .01 -> .0001
- link translation: mass .01 -> .0001
- link wheel1: mass 1.22527899288125 -> 1
- link wheel2: mass 1.22527899288124 -> 1
- link wheel3: mass 1.22527899288124 -> 1
- link wheel4: mass 1.22527899288125 -> 1
Joints:
- joint camera_joint: origin xyz=0 0.2 0.45 rpy=0 0 3.14 -> xyz=0 0.0 0.45 rpy=0 0 3.14
- joint joint_sensor_laser: origin xyz=1.05 0 0.5 rpy=0 0.0 0.0 -> xyz=1.05 0 0.4 rpy=0 0.5 0.0

Commit message: Created custom odom and transform publishder to publish transform based on gazebo model state instead of diff drive controller

File: src/FullMech_Rep/urdf/FullMech_Rep.urdf (robot description, URDF)
Before this commit: robot FullMech_Rep, 11 links, 10 joints
Joints:
- joint joint_sensor_laser: origin xyz=1.05 0 0.4 rpy=0 0.5 0.0 -> xyz=1.05 0 0.4 rpy=0 0.0 0.0

Commit message: Turned down mass value of wheels to improve autonmous navigation performance. Tuned param files for move_base

File: src/FullMech_Rep/urdf/FullMech_Rep.urdf (robot description, URDF)
Before this commit: robot FullMech_Rep, 11 links, 10 joints
Links:
- link sensor_laser: mass .0001 -> .000001
- link wheel1: mass 1 -> 0.1
- link wheel2: mass 1 -> 0.1
- link wheel3: mass 1 -> 0.1
- link wheel4: mass 1 -> 0.1
